File: kicad/fakefire.kicad_sch (KiCad schematic)
At the start: 45 parts, among them J1 Barrel_Jack, J2 Conn_01x03_Female, J3 Left speaker, J4 Right speaker, Q2 IRLB3813PBF, U1 YAAJ_DCDC_StepDown_LM2596, U2 PAM8403_Module, U3 TSOP1838B, U4 DFR0299, U5 Raspberry Pico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

Commit message: update kicad files, added more infos, comments
Other:
- note added: "12V led strip control"
- note added: "Audio circuit"
- note added: "Barrel Jack, 5V and 4V generation with Power leds"
- note added: "Decoupling"
- note added: "IR reception & voltage conversion"
- note added: "Mounting holes (board/speaker)"
- note added: "NAND 3.3V conversion to 5V"
- company: (none) -> N/A
- title: (none) -> Fakefire Project
- moved on the sheet: D3, H1, H10, H2, H3, H4, H5, H6, H7, H8, H9, J3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
